Commit message: Imported upstream version '0.5.13' of 'upstream'

File: nao_description/urdf/naoV33_generated_urdf/nao_arms.xacro (robot description, xacro)
@@ -168,5 +168,5 @@
 		<parent link="r_wrist"/>
 		<child link="r_gripper"/>
-		<origin rpy="0 0 0" xyz="0.05775 0 -0.01213"/>
+		<origin rpy="0 0 0" xyz="0.05775 0 -0.01231"/>
 		<axis xyz="1.0 0 0"/>
 		<limit effort="0.292" lower="0" upper="1.0" velocity="8.33"/>

File: nao_description/urdf/naoV40_generated_urdf/nao_arms.xacro (robot description, xacro)
@@ -168,5 +168,5 @@
 		<parent link="r_wrist"/>
 		<child link="r_gripper"/>
-		<origin rpy="0 0 0" xyz="0.05775 0 -0.01213"/>
+		<origin rpy="0 0 0" xyz="0.05775 0 -0.01231"/>
 		<axis xyz="1.0 0 0"/>
 		<limit effort="0.292" lower="0" upper="1.0" velocity="8.33"/>

File: nao_description/urdf/naoV50_generated_urdf/nao_arms.xacro (robot description, xacro)
@@ -168,5 +168,5 @@
 		<parent link="r_wrist"/>
 		<child link="r_gripper"/>
-		<origin rpy="0 0 0" xyz="0.05775 0 -0.01213"/>
+		<origin rpy="0 0 0" xyz="0.05775 0 -0.01231"/>
 		<axis xyz="1.0 0 0"/>
 		<limit effort="0.292" lower="0" upper="1.0" velocity="8.33"/>
